File: processor.sch (KiCad schematic (older format))
At the start: 1 part

Commit message: Added decoupling capacitors to the processor schematic.
Parts:
- added C? (x2): 2.2uF, 0603, symbol C
- added C?: 4.7uF, 0805, symbol C
- added C? (x12): 100nF, 0603, symbol C
- added C?: 10nF, 0603, symbol C
- added C?: 1uF, 0603, symbol C
Connections:
- net labels added: AGND, DGND
- wire segments 0 -> 23
