File: connections.sch (KiCad schematic (older format))
At the start: 6 parts

Commit message: Re-arranged the connections schematic to make it a little more orginized
Other:
- note added: "RJ-45 Jack"
- note added: "microSD Card"
- note added: "microUSB Jack"
- moved on the sheet: J?, uSD?
Changed lines of the file:
@@
-EESchema Schematic File Version 2  date 9/27/2011 12:42:11 AM
+EESchema Schematic File Version 2  date 9/27/2011 6:56:40 AM
 LIBS:power
 LIBS:device
@@
 $Descr A4 11700 8267
 encoding utf-8
-Sheet 3 7
+Sheet 5 7
 Title "noname.sch"
 Date "27 sep 2011"
@@
 Comment4 ""
 $EndDescr
+Text Notes 5410 650  0    100  ~ 20
+RJ-45 Jack
+Wire Notes Line
+	7980 490  5380 490
+Wire Notes Line
+	7980 490  7980 1850
+Wire Notes Line
+	7980 1850 5380 1850
+Wire Notes Line
+	5380 1850 5380 490
+Wire Notes Line
+	3250 490  1360 490
+Wire Notes Line
+	3250 490  3250 1680
+Wire Notes Line
+	3250 1680 1360 1680
 Wire Wire Line
 	1250 1480 1250 1440
@@
 	650  840  650  940
 Wire Wire Line
-	3600 1250 3950 1250
-Wire Wire Line
-	3600 1350 3950 1350
-Wire Wire Line
-	3600 1450 3950 1450
-Wire Wire Line
-	3600 1550 3950 1550
-Wire Wire Line
-	3600 1650 3950 1650
-Wire Wire Line
-	3600 1750 3950 1750
-Wire Wire Line
-	3600 1850 3950 1850
-Wire Wire Line
-	3600 1950 3950 1950
+	2340 850  2690 850
+Wire Wire Line
+	2340 950  2690 950
+Wire Wire Line
+	2340 1050 2690 1050
+Wire Wire Line
+	2340 1150 2690 1150
+Wire Wire Line
+	2340 1250 2690 1250
+Wire Wire Line
+	2340 1350 2690 1350
+Wire Wire Line
+	2340 1450 2690 1450
+Wire Wire Line
+	2340 1550 2690 1550
 Wire Wire Line
 	1250 940  1250 840
@@
 Wire Notes Line
 	500  1590 1330 1590
+Wire Notes Line
+	1360 1680 1360 490
+Wire Notes Line
+	3280 1680 3280 490
+Wire Notes Line
+	3280 1680 5350 1680
+Wire Notes Line
+	5350 1680 5350 490
+Wire Notes Line
+	5350 490  3280 490
+Text Notes 3280 670  0    100  ~ 20
+microUSB Jack
+Text Notes 1400 700  0    100  ~ 20
+microSD Card
 Text Notes 540  700  0    100  ~ 20
 Reset
@@
 	1    0    0    -1
 $EndComp
-Text HLabel 3950 1950 2    60   Input ~ 0
+Text HLabel 2690 1550 2    60   Input ~ 0
 uSD_Data1
-Text HLabel 3950 1850 2    60   Input ~ 0
+Text HLabel 2690 1450 2    60   Input ~ 0
 uSD_Data0
 $Comp
 L DGND #PWR?
 U 1 1 4E8152D9
-P 3950 1750
+P 2690 1350
 AR Path="/4E7A8C23/4E7E0D6B/4E8152D9" Ref="#PWR?"  Part="1"
 AR Path="/4E7DF058/4E815305/4E8152D9" Ref="#PWR?"  Part="1"
 AR Path="/4E8158D9/4E8152D9" Ref="#PWR?"  Part="1"
 AR Path="/4E815C62/4E815C93/4E8152D9" Ref="#PWR?"  Part="1"
-F 0 "#PWR?" H 3950 1750 40  0001 C CNN
-F 1 "DGND" H 3950 1680 40  0000 C CNN
-	1    3950 1750
+F 0 "#PWR?" H 2690 1350 40  0001 C CNN
+F 1 "DGND" H 2690 1280 40  0000 C CNN
+	1    2690 1350
 	0    -1   -1   0
 $EndComp
-Text HLabel 3950 1650 2    60   Input ~ 0
+Text HLabel 2690 1250 2    60   Input ~ 0
 uSD_CLK
 $Comp
 L +3.3V #PWR?
 U 1 1 4E8152C3
-P 3950 1550
+P 2690 1150
 AR Path="/4E7A8C23/4E7E0D6B/4E8152C3" Ref="#PWR?"  Part="1"
 AR Path="/4E7DF058/4E815305/4E8152C3" Ref="#PWR?"  Part="1"
 AR Path="/4E8158D9/4E8152C3" Ref="#PWR?"  Part="1"
 AR Path="/4E815C62/4E815C93/4E8152C3" Ref="#PWR?"  Part="1"
-F 0 "#PWR?" H 3950 1510 30  0001 C CNN
-F 1 "+3.3V" H 3950 1660 30  0000 C CNN
-	1    3950 1550
+F 0 "#PWR?" H 2690 1110 30  0001 C CNN
+F 1 "+3.3V" H 2690 1260 30  0000 C CNN
+	1    2690 1150
 	0    1    1    0
 $EndComp
-Text HLabel 3950 1450 2    60   Input ~ 0
+Text HLabel 2690 1050 2    60   Input ~ 0
 uSD_CMD
-Text HLabel 3950 1350 2    60   Input ~ 0
+Text HLabel 2690 950  2    60   Input ~ 0
 uSD_Data3
-Text HLabel 3950 1250 2    60   Input ~ 0
+Text HLabel 2690 850  2    60   Input ~ 0
 uSD_Data2
 $Comp
 L MICROSD uSD?
 U 1 1 4E815102
-P 3000 1600
+P 1740 1200
 AR Path="/4E7A8C23/4E7E0D6B/4E815102" Ref="uSD?"  Part="1"
 AR Path="/4E7DF058/4E815305/4E815102" Ref="uSD?"  Part="1"
 AR Path="/4E8158D9/4E815102" Ref="uSD?"  Part="1"
 AR Path="/4E815C62/4E815C93/4E815102" Ref="uSD?"  Part="1"
-F 0 "uSD?" H 3000 1450 60  0000 C CNN
-F 1 "MICROSD" H 3000 1350 60  0000 C CNN
-	1    3000 1600
+F 0 "uSD?" H 1740 1050 60  0000 C CNN
+F 1 "MICROSD" H 1740 950 60  0000 C CNN
+	1    1740 1200
 	0    1    1    0
 $EndComp
-NoConn ~ 8100 2200
-NoConn ~ 8100 2100
-Text HLabel 8100 2000 0    60   Output ~ 0
+NoConn ~ 6140 1760
+NoConn ~ 6140 1660
+Text HLabel 6140 1560 0    60   Output ~ 0
 Phy_LedGreen-
-Text HLabel 8100 1900 0    60   Input ~ 0
+Text HLabel 6140 1460 0    60   Input ~ 0
 Phy_LedGreen+
 $Comp
 L DGND #PWR?
 U 1 1 4E7E1857
-P 8100 1800
+P 6140 1360
 AR Path="/4E7A8C23/4E7E0D6B/4E7E1857" Ref="#PWR?"  Part="1"
 AR Path="/4E7DF058/4E815305/4E7E1857" Ref="#PWR?"  Part="1"
 AR Path="/4E8158D9/4E7E1857" Ref="#PWR?"  Part="1"
 AR Path="/4E815C62/4E815C93/4E7E1857" Ref="#PWR?"  Part="1"
-F 0 "#PWR?" H 8100 1800 40  0001 C CNN
-F 1 "DGND" H 8100 1730 40  0000 C CNN
-	1    8100 1800
+F 0 "#PWR?" H 6140 1360 40  0001 C CNN
+F 1 "DGND" H 6140 1290 40  0000 C CNN
+	1    6140 1360
 	0    1    1    0
 $EndComp
-NoConn ~ 8100 1600
-NoConn ~ 8100 1600
-NoConn ~ 8100 1300
-NoConn ~ 8100 1300
-Text HLabel 8100 1700 0    60   BiDi ~ 0
+NoConn ~ 6140 1160
+NoConn ~ 6140 1160
+NoConn ~ 6140 860
+NoConn ~ 6140 860
+Text HLabel 6140 1260 0    60   BiDi ~ 0
 Phy_recv-
-Text HLabel 8100 1500 0    60   BiDi ~ 0
+Text HLabel 6140 1060 0    60   BiDi ~ 0
 Phy_recv+
-Text HLabel 8100 1400 0    60   BiDi ~ 0
+Text HLabel 6140 960  0    60   BiDi ~ 0
 Phy_trans-
-Text HLabel 8100 1200 0    60   BiDi ~ 0
+Text HLabel 6140 760  0    60   BiDi ~ 0
 Phy_trans+
 $Comp
 L GNDPWR #PWR?
 U 1 1 4E743F0C
-P 9800 2100
+P 7840 1660
 AR Path="/4E7A8C23/4E7E0D6B/4E743F0C" Ref="#PWR?"  Part="1"
 AR Path="/4E7DF058/4E815305/4E743F0C" Ref="#PWR?"  Part="1"
 AR Path="/4E8158D9/4E743F0C" Ref="#PWR?"  Part="1"
 AR Path="/4E815C62/4E815C93/4E743F0C" Ref="#PWR?"  Part="1"
-F 0 "#PWR?" H 9800 2150 40  0001 C CNN
-F 1 "GNDPWR" H 9800 2020 40  0000 C CNN
-	1    9800 2100
+F 0 "#PWR?" H 7840 1710 40  0001 C CNN
+F 1 "GNDPWR" H 7840 1580 40  0000 C CNN
+	1    7840 1660
 	1    0    0    -1
 $EndComp
@@
 L +5V #PWR?
 U 1 1 4E743DEE
-P 5550 1600
+P 3720 1130
 AR Path="/4E7A8C23/4E7E0D6B/4E743DEE" Ref="#PWR?"  Part="1"
 AR Path="/4E7DF058/4E815305/4E743DEE" Ref="#PWR?"  Part="1"
 AR Path="/4E8158D9/4E743DEE" Ref="#PWR?"  Part="1"
 AR Path="/4E815C62/4E815C93/4E743DEE" Ref="#PWR?"  Part="1"
-F 0 "#PWR?" H 5550 1690 20  0001 C CNN
-F 1 "+5V" H 5550 1690 30  0000 C CNN
-	1    5550 1600
+F 0 "#PWR?" H 3720 1220 20  0001 C CNN
+F 1 "+5V" H 3720 1220 30  0000 C CNN
+	1    3720 1130
 	1    0    0    -1
 $EndComp
@@
 L GNDPWR #PWR?
 U 1 1 4E743D61
-P 5550 2000
+P 3720 1530
 AR Path="/4E7A8C23/4E7E0D6B/4E743D61" Ref="#PWR?"  Part="1"
 AR Path="/4E7DF058/4E815305/4E743D61" Ref="#PWR?"  Part="1"
 AR Path="/4E8158D9/4E743D61" Ref="#PWR?"  Part="1"
 AR Path="/4E815C62/4E815C93/4E743D61" Ref="#PWR?"  Part="1"
-F 0 "#PWR?" H 5550 2050 40  0001 C CNN
-F 1 "GNDPWR" H 5550 1920 40  0000 C CNN
-	1    5550 2000
+F 0 "#PWR?" H 3720 1580 40  0001 C CNN
+F 1 "GNDPWR" H 3720 1450 40  0000 C CNN
+	1    3720 1530
 	1    0    0    -1
 $EndComp
@@
 L GNDPWR #PWR?
 U 1 1 4E743D59
-P 7050 1800
+P 5220 1330
 AR Path="/4E7A8C23/4E7E0D6B/4E743D59" Ref="#PWR?"  Part="1"
 AR Path="/4E7DF058/4E815305/4E743D59" Ref="#PWR?"  Part="1"
 AR Path="/4E8158D9/4E743D59" Ref="#PWR?"  Part="1"
 AR Path="/4E815C62/4E815C93/4E743D59" Ref="#PWR?"  Part="1"
-F 0 "#PWR?" H 7050 1850 40  0001 C CNN
-F 1 "GNDPWR" H 7050 1720 40  0000 C CNN
-	1    7050 1800
+F 0 "#PWR?" H 5220 1380 40  0001 C CNN
+F 1 "GNDPWR" H 5220 1250 40  0000 C CNN
+	1    5220 1330
 	1    0    0    -1
 $EndComp
@@
 L MICROUSB uUSB?
 U 1 1 4E743BB6
-P 6300 1800
+P 4470 1330
 AR Path="/4E7A8C23/4E7E0D6B/4E743BB6" Ref="uUSB?"  Part="1"
 AR Path="/4E7DF058/4E815305/4E743BB6" Ref="uUSB?"  Part="1"
 AR Path="/4E8158D9/4E743BB6" Ref="uUSB?"  Part="1"
 AR Path="/4E815C62/4E815C93/4E743BB6" Ref="uUSB?"  Part="1"
-F 0 "uUSB?" H 6300 2150 50  0000 C CNN
-F 1 "MICROUSB" H 6500 1600 50  0000 C CNN
-	1    6300 1800
+F 0 "uUSB?" H 4470 1680 50  0000 C CNN
+F 1 "MICROUSB" H 4670 1130 50  0000 C CNN
+	1    4470 1330
 	1    0    0    -1
 $EndComp
@@
 L RJ45-TRANSFO J?
 U 1 1 4E741312
-P 9200 1700
+P 7240 1260
 AR Path="/4E7A8C23/4E7E0D6B/4E741312" Ref="J?"  Part="1"
 AR Path="/4E7DF058/4E815305/4E741312" Ref="J?"  Part="1"
 AR Path="/4E8158D9/4E741312" Ref="J?"  Part="1"
 AR Path="/4E815C62/4E815C93/4E741312" Ref="J?"  Part="1"
-F 0 "J?" H 9300 2300 60  0000 L CNN
-F 1 "RJ45-TRANSFO" H 9150 2300 60  0000 R CNN
-	1    9200 1700
-	1    0    0    -1
-$EndComp
+F 0 "J?" H 7340 1860 60  0000 L CNN
+F 1 "RJ45-TRANSFO" H 7190 1860 60  0000 R CNN
+	1    7240 1260
+	1    0    0    -1
+$EndComp
