File: connections.sch (KiCad schematic (older format))
At the start: 6 parts

Commit message: Added some more of the connectors to the Dev Board.  Will work through the camera, spi, i2c and cans interfaces next
Other:
- note added: "DCMI Camera Conn"
Changed lines of the file:
@@
-EESchema Schematic File Version 2  date 10/15/2011 10:14:08 AM
+EESchema Schematic File Version 2  date 10/16/2011 9:20:50 PM
 LIBS:power
 LIBS:device
@@
 $Descr A4 11700 8267
 encoding utf-8
-Sheet 5 8
+Sheet 3 9
 Title "noname.sch"
-Date "15 oct 2011"
+Date "16 oct 2011"
 Rev ""
 Comp ""
@@
 Comment4 ""
 $EndDescr
+Text Notes 8050 650  0    100  ~ 20
+DCMI Camera Conn
+Wire Notes Line
+	8000 1850 8000 500
+Wire Notes Line
+	8000 1850 11200 1850
+Wire Notes Line
+	11200 1850 11200 500
+Wire Notes Line
+	11200 500  8000 500
+Wire Notes Line
+	5350 490  3280 490
+Wire Notes Line
+	5350 490  5350 1680
+Wire Notes Line
+	5350 1680 3280 1680
+Wire Notes Line
+	3280 1680 3280 490
+Wire Notes Line
+	1360 1680 1360 490
+Wire Notes Line
+	500  1590 1330 1590
+Wire Notes Line
+	500  1590 500  490
+Wire Notes Line
+	500  490  1330 490
+Wire Notes Line
+	1330 490  1330 1590
+Wire Wire Line
+	1250 940  1250 840
+Wire Wire Line
+	2340 1550 2690 1550
+Wire Wire Line
+	2340 1450 2690 1450
+Wire Wire Line
+	2340 1350 2690 1350
+Wire Wire Line
+	2340 1250 2690 1250
+Wire Wire Line
+	2340 1150 2690 1150
+Wire Wire Line
+	2340 1050 2690 1050
+Wire Wire Line
+	2340 950  2690 950
+Wire Wire Line
+	2340 850  2690 850
+Wire Wire Line
+	650  840  650  940
+Wire Wire Line
+	550  890  650  890
+Connection ~ 650  890
+Wire Wire Line
+	1250 1480 1250 1440
+Wire Notes Line
+	1360 1680 3250 1680
+Wire Notes Line
+	3250 1680 3250 490
+Wire Notes Line
+	3250 490  1360 490
+Wire Notes Line
+	5380 1850 5380 490
+Wire Notes Line
+	5380 1850 7980 1850
+Wire Notes Line
+	7980 1850 7980 490
+Wire Notes Line
+	7980 490  5380 490
 Text Notes 5410 650  0    100  ~ 20
 RJ-45 Jack
-Wire Notes Line
-	7980 490  5380 490
-Wire Notes Line
-	7980 490  7980 1850
-Wire Notes Line
-	7980 1850 5380 1850
-Wire Notes Line
-	5380 1850 5380 490
-Wire Notes Line
-	3250 490  1360 490
-Wire Notes Line
-	3250 490  3250 1680
-Wire Notes Line
-	3250 1680 1360 1680
-Wire Wire Line
-	1250 1480 1250 1440
-Connection ~ 650  890
-Wire Wire Line
-	550  890  650  890
-Wire Wire Line
-	650  840  650  940
-Wire Wire Line
-	2340 850  2690 850
-Wire Wire Line
-	2340 950  2690 950
-Wire Wire Line
-	2340 1050 2690 1050
-Wire Wire Line
-	2340 1150 2690 1150
-Wire Wire Line
-	2340 1250 2690 1250
-Wire Wire Line
-	2340 1350 2690 1350
-Wire Wire Line
-	2340 1450 2690 1450
-Wire Wire Line
-	2340 1550 2690 1550
-Wire Wire Line
-	1250 940  1250 840
-Wire Notes Line
-	1330 490  1330 1590
-Wire Notes Line
-	1330 490  500  490
-Wire Notes Line
-	500  490  500  1590
-Wire Notes Line
-	500  1590 1330 1590
-Wire Notes Line
-	1360 1680 1360 490
-Wire Notes Line
-	3280 1680 3280 490
-Wire Notes Line
-	3280 1680 5350 1680
-Wire Notes Line
-	5350 1680 5350 490
-Wire Notes Line
-	5350 490  3280 490
 Text Notes 3280 670  0    100  ~ 20
 microUSB Jack
@@
 AR Path="/4E7A8C23/4E7E0D6B/4E815BB9" Ref="#PWR?"  Part="1"
 AR Path="/4E815C62/4E815C93/4E815BB9" Ref="#PWR?"  Part="1"
+AR Path="/4E98DB6D/4E99DCE6/4E815BB9" Ref="#PWR?"  Part="1"
+AR Path="/4E7DF058/4E815305/4E815BB9" Ref="#PWR?"  Part="1"
 F 0 "#PWR?" H 650 1400 30  0001 C CNN
 F 1 "+3.3V" H 650 1550 30  0000 C CNN
@@
 AR Path="/4E7A8C23/4E7E0D6B/4E815A3B" Ref="SW?"  Part="1"
 AR Path="/4E815C62/4E815C93/4E815A3B" Ref="SW?"  Part="1"
+AR Path="/4E98DB6D/4E99DCE6/4E815A3B" Ref="SW?"  Part="1"
+AR Path="/4E7DF058/4E815305/4E815A3B" Ref="SW?"  Part="1"
 F 0 "SW?" H 1100 950 50  0000 C CNN
 F 1 "SW_PUSH" H 950 760 50  0000 C CNN
@@
 AR Path="/4E7A8C23/4E7E0D6B/4E815B81" Ref="R?"  Part="1"
 AR Path="/4E815C62/4E815C93/4E815B81" Ref="R?"  Part="1"
+AR Path="/4E98DB6D/4E99DCE6/4E815B81" Ref="R?"  Part="1"
+AR Path="/4E7DF058/4E815305/4E815B81" Ref="R?"  Part="1"
 F 0 "R?" V 1330 1190 50  0000 C CNN
 F 1 "1k" V 1250 1190 50  0000 C CNN
@@
 AR Path="/4E7A8C23/4E7E0D6B/4E815AE8" Ref="R?"  Part="1"
 AR Path="/4E815C62/4E815C93/4E815AE8" Ref="R?"  Part="1"
+AR Path="/4E98DB6D/4E99DCE6/4E815AE8" Ref="R?"  Part="1"
+AR Path="/4E7DF058/4E815305/4E815AE8" Ref="R?"  Part="1"
 F 0 "R?" V 730 1190 50  0000 C CNN
 F 1 "10k" V 650 1190 50  0000 C CNN
@@
 AR Path="/4E7A8C23/4E7E0D6B/4E815A9A" Ref="#PWR?"  Part="1"
 AR Path="/4E815C62/4E815C93/4E815A9A" Ref="#PWR?"  Part="1"
+AR Path="/4E98DB6D/4E99DCE6/4E815A9A" Ref="#PWR?"  Part="1"
+AR Path="/4E7DF058/4E815305/4E815A9A" Ref="#PWR?"  Part="1"
 F 0 "#PWR?" H 1250 1480 40  0001 C CNN
 F 1 "DGND" H 1250 1410 40  0000 C CNN
@@
 AR Path="/4E8158D9/4E8152D9" Ref="#PWR?"  Part="1"
 AR Path="/4E815C62/4E815C93/4E8152D9" Ref="#PWR?"  Part="1"
+AR Path="/4E98DB6D/4E99DCE6/4E8152D9" Ref="#PWR?"  Part="1"
 F 0 "#PWR?" H 2690 1350 40  0001 C CNN
 F 1 "DGND" H 2690 1280 40  0000 C CNN
@@
 AR Path="/4E8158D9/4E8152C3" Ref="#PWR?"  Part="1"
 AR Path="/4E815C62/4E815C93/4E8152C3" Ref="#PWR?"  Part="1"
+AR Path="/4E98DB6D/4E99DCE6/4E8152C3" Ref="#PWR?"  Part="1"
 F 0 "#PWR?" H 2690 1110 30  0001 C CNN
 F 1 "+3.3V" H 2690 1260 30  0000 C CNN
@@
 AR Path="/4E8158D9/4E815102" Ref="uSD?"  Part="1"
 AR Path="/4E815C62/4E815C93/4E815102" Ref="uSD?"  Part="1"
+AR Path="/4E98DB6D/4E99DCE6/4E815102" Ref="uSD?"  Part="1"
 F 0 "uSD?" H 1740 1050 60  0000 C CNN
 F 1 "MICROSD" H 1740 950 60  0000 C CNN
@@
 AR Path="/4E8158D9/4E7E1857" Ref="#PWR?"  Part="1"
 AR Path="/4E815C62/4E815C93/4E7E1857" Ref="#PWR?"  Part="1"
+AR Path="/4E98DB6D/4E99DCE6/4E7E1857" Ref="#PWR?"  Part="1"
 F 0 "#PWR?" H 6140 1360 40  0001 C CNN
 F 1 "DGND" H 6140 1290 40  0000 C CNN
@@
 AR Path="/4E8158D9/4E743F0C" Ref="#PWR?"  Part="1"
 AR Path="/4E815C62/4E815C93/4E743F0C" Ref="#PWR?"  Part="1"
+AR Path="/4E98DB6D/4E99DCE6/4E743F0C" Ref="#PWR?"  Part="1"
 F 0 "#PWR?" H 7840 1710 40  0001 C CNN
 F 1 "GNDPWR" H 7840 1580 40  0000 C CNN
@@
 AR Path="/4E8158D9/4E743DEE" Ref="#PWR?"  Part="1"
 AR Path="/4E815C62/4E815C93/4E743DEE" Ref="#PWR?"  Part="1"
+AR Path="/4E98DB6D/4E99DCE6/4E743DEE" Ref="#PWR?"  Part="1"
 F 0 "#PWR?" H 3720 1220 20  0001 C CNN
 F 1 "+5V" H 3720 1220 30  0000 C CNN
@@
 AR Path="/4E8158D9/4E743D61" Ref="#PWR?"  Part="1"
 AR Path="/4E815C62/4E815C93/4E743D61" Ref="#PWR?"  Part="1"
+AR Path="/4E98DB6D/4E99DCE6/4E743D61" Ref="#PWR?"  Part="1"
 F 0 "#PWR?" H 3720 1580 40  0001 C CNN
 F 1 "GNDPWR" H 3720 1450 40  0000 C CNN
@@
 AR Path="/4E8158D9/4E743D59" Ref="#PWR?"  Part="1"
 AR Path="/4E815C62/4E815C93/4E743D59" Ref="#PWR?"  Part="1"
+AR Path="/4E98DB6D/4E99DCE6/4E743D59" Ref="#PWR?"  Part="1"
 F 0 "#PWR?" H 5220 1380 40  0001 C CNN
 F 1 "GNDPWR" H 5220 1250 40  0000 C CNN
@@
 AR Path="/4E8158D9/4E743BB6" Ref="uUSB?"  Part="1"
 AR Path="/4E815C62/4E815C93/4E743BB6" Ref="uUSB?"  Part="1"
+AR Path="/4E98DB6D/4E99DCE6/4E743BB6" Ref="uUSB?"  Part="1"
 F 0 "uUSB?" H 4470 1680 50  0000 C CNN
 F 1 "MICROUSB" H 4670 1130 50  0000 C CNN
@@
 AR Path="/4E8158D9/4E741312" Ref="J?"  Part="1"
 AR Path="/4E815C62/4E815C93/4E741312" Ref="J?"  Part="1"
+AR Path="/4E98DB6D/4E99DCE6/4E741312" Ref="J?"  Part="1"
 F 0 "J?" H 7340 1860 60  0000 L CNN
 F 1 "RJ45-TRANSFO" H 7190 1860 60  0000 R CNN
